File: pro/hardware/kicad/v1/Dreamstalker-PRO-v1/Dreamstalker-PRO-v1.kicad_pcb (KiCad board)
At the start: 2 copper layers, 68 parts, among them J1 Header 2x3, J2 Header 2x5, J3 ST-033, J4 CSCONN T-Flash Card, Q1 IRLML2402, Q2 BC807-40, Q3 BC807-40, Q4 BC807-40, Q5 BC807-40, Q6 KP-3216P3C, SW1 SELECT, SW2 ENTER, SW3 POWER, SW4 CHECK, SW5 [+], SW6 [-], U1 ATmega128L-8AI, U2 MC34119D, U3 VS1002D, Y1 32768 KHz, Y2 12.0 MHz

Commit message: Planned update
Parts:
- added BT1: BH421-3A, Dreamstalker-Footprints:BatteryHolder_BH421-3A, F.Cu at (127.4, 84.0)
- added C14: 10u, Dreamstalker-Footprints:CP_EIA-3216-18_Kemet-A, B.Cu at (153.1, 47.4)
- added C15: 4.7u, Dreamstalker-Footprints:C_0805_2012Metric, F.Cu at (110.3, 116.4)
- added C16: 1u, Dreamstalker-Footprints:C_0805_2012Metric, B.Cu at (147.5, 47.2)
- added C17: 1u, Dreamstalker-Footprints:C_0805_2012Metric, B.Cu at (147.6, 44.1)
- added C18: 1u, Dreamstalker-Footprints:C_0805_2012Metric, B.Cu at (147.5, 50.4)
- added C19: 22n, Dreamstalker-Footprints:C_0805_2012Metric, F.Cu at (104.2, 117.3)
- added C20: 4.7u, Dreamstalker-Footprints:C_0805_2012Metric, F.Cu at (101.8, 117.3)
- added D4: 1N5819, Dreamstalker-Footprints:D_SOD-123, F.Cu at (104.5, 120.7)
- added M1: Vibration Motor, Dreamstalker-Footprints:VIBRO-MOTOR_SMD, F.Cu at (95.5, 82.3)
- added R26: 100, Dreamstalker-Footprints:R_0603_1608Metric, F.Cu at (141.4, 54.0)
- added R27: 10K, Dreamstalker-Footprints:R_0603_1608Metric, B.Cu at (143.2, 44.3)
- added REF**: KiCad-Logo2_6mm_SilkScreen, Symbol:KiCad-Logo2_6mm_SilkScreen, B.Cu at (160.2, 121.2)
- added U4: RT9193-33GB, Dreamstalker-Footprints:SOT94P279X130-5N, F.Cu at (107.2, 116.8)
- C10, C13, C2, C3, C6, C8, R1, R10, R11, R12, R13, R14, R15, R16, R19, R20, R21, R22, R23, R24, R4, R5, R7, R8, R9, U2, Y1: moved to B.Cu
- C4: value 0.1u -> 1u; moved to B.Cu
- C5: value 47u -> 22u; moved to B.Cu
- D1, D2, D3: footprint Dreamstalker-Footprints:LEDC3216X110N -> Dreamstalker-Footprints:LEDC3216X110N-TH
- Q6: footprint Dreamstalker-Footprints:LEDC3216X130N -> Dreamstalker-Footprints:LEDC3216X130N-TH
- R17, R18: value 240 -> 10K; moved to B.Cu
- R6: value 4.7K -> 10K; moved to B.Cu
- moved U2 133.6 mm to (158.6, 47.4), turned to 180 degrees
- moved C6 106.3 mm to (138.3, 56.5), turned to 180 degrees
- moved R13 100.2 mm to (162.7, 116.0)
- moved R20 97.8 mm to (147.7, 59.7), turned to 90 degrees
- moved C4 97.6 mm to (163.7, 55.6), turned to 270 degrees
- moved C5 97.3 mm to (163.7, 60.4), turned to 90 degrees
- moved R15 95.9 mm to (157.5, 68.2)
- moved R19 94.3 mm to (153.8, 53.0), turned to 180 degrees
- moved R7 91.8 mm to (153.3, 60.0), turned to 270 degrees
- moved C3 90.1 mm to (137.4, 100.4), turned to 270 degrees
- moved D2 88.3 mm to (162.8, 110.3)
- moved C2 86.6 mm to (155.8, 60.1), turned to 90 degrees
- moved R4 85.8 mm to (158.3, 65.4), turned to 90 degrees
- moved R8 81.2 mm to (158.3, 71.0)
- moved R21 80.5 mm to (149.9, 71.2), turned to 90 degrees
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Connections:
- J2 pad 7: Net-(J2-Pad7) -> +5V
- J3 pad R: Net-(J3-PadR) -> /HPR
- J3 pad T: Net-(J3-PadT) -> /HPL
- J4 pad 2: /CDCS -> /SDCS
- R17 pad 1: /HPR -> Net-(C16-Pad2)
- R17 pad 2: Net-(J3-PadR) -> /HPR
- R18 pad 1: /HPL -> Net-(C18-Pad2)
- R18 pad 2: Net-(J3-PadT) -> /HPL
- R24 pad 1: /CDCS -> /SDCS
Routing:
- net GND: track 43.6 -> 561.4 mm, vias 1 -> 62
- net +3V: track 29.7 -> 484.6 mm, vias 7 -> 19
- net /RESET: track 0.00 -> 135.0 mm
- net /HPR: track 0.00 -> 106.3 mm
- net /SNDOFF: track 0.00 -> 88.3 mm, vias 0 -> 2
- net /HPL: track 0.00 -> 86.1 mm, vias 0 -> 4
- net /SOUND: track 0.00 -> 83.0 mm, vias 0 -> 2
- net /GBUF: track 0.00 -> 82.9 mm, vias 0 -> 2
- net /IRRX: track 0.00 -> 82.8 mm, vias 0 -> 1
- net /SCK: track 0.00 -> 76.5 mm, vias 0 -> 3
- net /LED2: track 0.00 -> 76.5 mm, vias 0 -> 3
- net /KEY6: track 2.30 -> 74.9 mm
- net /XCS: track 0.00 -> 71.7 mm, vias 0 -> 2
- net /HPTS: track 0.00 -> 66.8 mm, vias 0 -> 2
- net /PDI: track 0.00 -> 66.3 mm, vias 0 -> 1
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- added copper zone on B.Cu, net GND
- added copper zone on F.Cu, net GND
Other:
- board outline added: 79 x 85 mm
- board text added: "-= DreamStalker PRO =-"
- board text added: "This side away from face"
