File: pro/hardware/kicad/v1/Dreamstalker-PRO-v1/Dreamstalker-PRO-v1.sch (KiCad schematic (older format))
At the start: 70 parts, among them J1 Header 2x3, J2 Header 2x5, J3 ST-033, J4 CSCONN T-Flash Card, M1 Vibration Motor, Q1 IRLML2402, Q2 BC807-40, Q3 BC807-40, Q4 BC807-40, Q5 BC807-40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

Commit message: Planned update
Parts:
- added C14: 10u, Dreamstalker-Footprints:CP_EIA-3216-18_Kemet-A, symbol Dreamstalker-Components:CP_Small
- added C15, C20: 4.7u, Dreamstalker-Footprints:C_0805_2012Metric, symbol Dreamstalker-Components:C_Small
- added C16, C17, C18: 1u, Dreamstalker-Footprints:C_0805_2012Metric, symbol Dreamstalker-Components:C_Small
- added C19: 22n, Dreamstalker-Footprints:C_0805_2012Metric, symbol Dreamstalker-Components:C_Small
- added D4: 1N5819, Dreamstalker-Footprints:D_SOD-123, symbol Dreamstalker-Components:D_Schottky
- added R26: 100, Dreamstalker-Footprints:R_0603_1608Metric, symbol Dreamstalker-Components:R_Small
- added R27: 10K, Dreamstalker-Footprints:R_0603_1608Metric, symbol Dreamstalker-Components:R_Small
- added U4: RT9193-33GB, Dreamstalker-Footprints:SOT94P279X130-5N, symbol Dreamstalker-Components:RT9193-33GB
- BT1: footprint (none) -> Dreamstalker-Footprints:BatteryHolder_BH421-3A
- C4: value 0.1u -> 1u
- C5: value 47u -> 22u
- D1, D2, D3: footprint Dreamstalker-Footprints:LEDC3216X110N -> Dreamstalker-Footprints:LEDC3216X110N-TH
- M1: footprint (none) -> Dreamstalker-Footprints:VIBRO-MOTOR_SMD
- Q6: footprint Dreamstalker-Footprints:LEDC3216X130N -> Dreamstalker-Footprints:LEDC3216X130N-TH
- R17, R18: value 240 -> 10K
- R6: value 4.7K -> 10K
Connections:
- net CDCS is gone; now on net SDCS: J4.2 (DAT3/CD), R24.1
- net +3V: now also C14.1, D4.1 (K)
- net GBUF: now also R27.2
- net GND: now also C14.2, C15.2, C16.1, C17.1, C18.1, C19.2, C20.2, U4.2 (GND)
- net HPL: now also J3.T, R18.2; no longer R18.1
- net HPR: now also J3.R, R17.2; no longer R17.1
- net SILENT: now also R26.1
- net +5V: now reaches J2.7 (Pin_7)
- net +5V: now also C15.1, U4.1 (VIN), U4.3 (EN)
- net at C5.1, U2.2 (FC2): now also R26.2
- new net: C19.1, U4.4 (BP)
- new net: C20.1, D4.2 (A), U4.5 (VOUT)
- new net: C18.2, R18.1
- new net: C16.2, R17.1
- new net: C17.2, R27.1
Other:
- moved on the sheet: C2, C4, DS1, J3, R1, R10, R15, R16, R19, R4, R5, R6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
