File: hardware/kicad/Ultra/Dreamstalker-Ultra-v1/Dreamstalker-Ultra-v1.sch (KiCad schematic (older format))
At the start: 81 parts, among them J1 Mini-USB-B, J2 PDI connector, J3 PJ-313D, J4 Speaker, J5 Battery, J6 ATTEND_112J-TDAR-R01, M1 Vibration Motor, Q1 KP-3216P3C, Q2 IRLML2402, Q3 IRLML6402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

Commit message: Dreamstalker-PRO PCB improvements
Parts:
- C14: value 1u -> 2.2u
Other:
- moved on the sheet: C18, C22, C4, J6, R1, R2, R21, R27, R3, SW1, SW2, SW3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
