File: hardware/kicad/PRO/Dreamstalker-PRO-v1/Dreamstalker-PRO-v1.kicad_pcb (KiCad board)
At the start: 2 copper layers, 79 x 85 mm, 76 parts, among them J1 Header 2x3, J2 Header 2x5, J3 ST-033, J4 ATTEND_112J-TDAR-R01, M1 Vibration Motor, Q1 IRLML2402, Q2 BC807-40, Q3 BC807-40, Q4 BC807-40, Q5 BC807-40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

Commit message: Dreamstalker-PRO PCB improvements
Parts:
- added C15: 10u, Dreamstalker-Footprints:CP_EIA-3216-18_Kemet-A, B.Cu at (142.2, 58.1)
- added R24: 100K, Dreamstalker-Footprints:R_0603_1608Metric, B.Cu at (147.5, 75.4)
- added R28: 100K, Dreamstalker-Footprints:R_0603_1608Metric, B.Cu at (149.2, 75.4)
- added R30: 100K, Dreamstalker-Footprints:R_0603_1608Metric, B.Cu at (143.6, 88.8)
- added R31: 100K, Dreamstalker-Footprints:R_0603_1608Metric, B.Cu at (143.6, 90.4)
- C13: value 0.1u -> 100n
- C16, C17, C18: value 1u -> 10n
- J1: value Header 2x3 -> UART Header
- J2: value Header 2x5 -> JTAG Header
- R17, R18, R27: value 10K -> 22
- R2: value 150 -> 0
- R3: value 47K -> 100K
- U1: value ATMEGA128L-8AI -> ATMEGA128L-8AU
- Y2: value 12.0 MHz -> 12.288M
- moved R2 7.09 mm to (91.3, 83.3), turned to 270 degrees
- moved R22 0.46 mm to (144.1, 57.4), turned to 90 degrees
Connections:
- C6 pad 2: Net-(C6-Pad2) -> Net-(C15-Pad1)
- M1 pad 1: +3V -> Net-(M1-Pad1)
- Q1 pad 1: Net-(Q1-Pad1) -> /VIBRO
- R2 pad 1: /VIBRO -> Net-(M1-Pad1)
- R2 pad 2: Net-(Q1-Pad1) -> +3V
- R20 pad 2: Net-(C6-Pad2) -> Net-(C15-Pad1)
- R22 pad 1: Net-(C6-Pad2) -> Net-(C7-Pad1)
- R22 pad 2: Net-(C7-Pad1) -> Net-(C15-Pad1)
- U3 pad 10: GND -> Net-(R28-Pad2)
- U3 pad 11: GND -> Net-(U3-Pad11)
- U3 pad 12: GND -> Net-(U3-Pad12)
- U3 pad 24: +3V -> Net-(U3-Pad24)
- U3 pad 25: GND -> Net-(U3-Pad25)
- U3 pad 31: +3V -> Net-(U3-Pad31)
- U3 pad 33: GND -> Net-(R31-Pad2)
- U3 pad 34: GND -> Net-(R30-Pad2)
- U3 pad 35: GND -> Net-(U3-Pad35)
- U3 pad 36: GND -> Net-(U3-Pad36)
- U3 pad 5: +3V -> Net-(U3-Pad5)
- U3 pad 7: +3V -> Net-(U3-Pad7)
- U3 pad 9: GND -> Net-(R24-Pad2)
Routing:
- net GND: track 560.4 -> 572.9 mm, vias 96 -> 98
- net Net-(C15-Pad1): track 0.00 -> 9.58 mm
- net Net-(C6-Pad2): track 9.52 -> 0.00 mm
- net +3V: track 483.6 -> 474.2 mm
- net /VIBRO: track 20.4 -> 27.9 mm
- net Net-(Q1-Pad1): track 5.32 -> 0.00 mm
- net Net-(R31-Pad2): track 0.00 -> 4.80 mm
- net /KEY1: track 48.5 -> 51.4 mm
- net Net-(R30-Pad2): track 0.00 -> 2.76 mm
- net /KEY2: track 54.0 -> 56.7 mm
- net Net-(M1-Pad1): track 0.00 -> 2.46 mm
- net Net-(R24-Pad2): track 0.00 -> 2.30 mm
- net Net-(R28-Pad2): track 0.00 -> 2.25 mm
- net /HPL: track 84.5 -> 85.9 mm
- net Net-(C7-Pad1): track 38.5 -> 39.8 mm
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
Commit message: Planned update
Parts:
- added C19: 10n, Dreamstalker-Footprints:C_0805_2012Metric, B.Cu at (134.1, 71.2)
- added C20: 10n, Dreamstalker-Footprints:C_0805_2012Metric, B.Cu at (144.6, 71.0)
- added C21: 0.1u, Dreamstalker-Footprints:C_0805_2012Metric, B.Cu at (120.4, 93.1)
- added L1: L_Small, Dreamstalker-Footprints:L_0805_2012Metric, B.Cu at (153.8, 74.7)
- added R29: 470, Dreamstalker-Footprints:R_0603_1608Metric, B.Cu at (140.6, 74.6)
- added R32: 470, Dreamstalker-Footprints:R_0603_1608Metric, B.Cu at (137.1, 74.6)
- C13: value 100n -> 1u
- C17: value 10n -> 47n
- C6: footprint Dreamstalker-Footprints:C_0805_2012Metric -> Dreamstalker-Footprints:CP_EIA-3216-18_Kemet-A
- R17, R18: value 22 -> 20
- R27: value 22 -> 10
- moved C6 1.33 mm to (137.2, 55.2), turned to 180 degrees
- moved C13 0.47 mm to (136.4, 84.8), turned to 0 degrees
- moved R7 0.17 mm to (153.5, 60.0)
Connections:
- C6 pad 1: Net-(C6-Pad1) -> Net-(C15-Pad1)
- C6 pad 2: Net-(C15-Pad1) -> Net-(C6-Pad2)
- J4 pad 9: Net-(J4-Pad9) -> /CD
- R21 pad 2: Net-(C6-Pad1) -> Net-(C6-Pad2)
- R23 pad 1: Net-(C6-Pad1) -> Net-(C6-Pad2)
- U1 pad 38: Net-(U1-Pad38) -> /CD
- U1 pad 62: Net-(U1-Pad62) -> /AREF
- U3 pad 1: Net-(C7-Pad2) -> Net-(C20-Pad1)
- U3 pad 11: Net-(U3-Pad11) -> GND
- U3 pad 12: Net-(U3-Pad12) -> GND
- U3 pad 14: +3V -> /VSVDD
- U3 pad 19: +3V -> /VSVDD
- U3 pad 2: Net-(C8-Pad2) -> Net-(C19-Pad2)
- U3 pad 24: Net-(U3-Pad24) -> /VSVDD
- U3 pad 25: Net-(U3-Pad25) -> GND
- U3 pad 26: +3V -> /VSVDD
- U3 pad 31: Net-(U3-Pad31) -> /VSVDD
- U3 pad 32: +3V -> /VSVDD
- U3 pad 35: Net-(U3-Pad35) -> GND
- U3 pad 36: Net-(U3-Pad36) -> GND
- U3 pad 38: +3V -> /VSVDD
- U3 pad 43: +3V -> /VSVDD
- U3 pad 45: +3V -> /VSVDD
- U3 pad 5: Net-(U3-Pad5) -> /VSVDD
- U3 pad 6: +3V -> /VSVDD
- U3 pad 7: Net-(U3-Pad7) -> /VSVDD
Routing:
- net /CD: track 0.00 -> 74.4 mm, vias 0 -> 2
- net /VSVDD: track 0.00 -> 41.9 mm
- net GND: track 572.9 -> 603.4 mm, vias 98 -> 110
- net Net-(C6-Pad1): track 28.0 -> 0.00 mm, vias 2 -> 0
- net Net-(C6-Pad2): track 0.00 -> 27.4 mm, vias 0 -> 2
- net +3V: track 474.2 -> 448.5 mm, vias 19 -> 20
- net Net-(C19-Pad2): track 0.00 -> 21.1 mm
- net Net-(C20-Pad1): track 0.00 -> 16.7 mm
- net Net-(C8-Pad2): track 17.0 -> 7.52 mm
- net Net-(C13-Pad2): track 16.5 -> 7.71 mm
- net /AREF: track 0.00 -> 8.61 mm
- net /HPR: track 105.5 -> 99.5 mm, vias 0 -> 2
- net Net-(C7-Pad2): track 11.5 -> 9.23 mm
- net /HPL: track 85.9 -> 88.1 mm
- net /SEGC: track 26.3 -> 28.2 mm
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