File: hardware/kicad/PRO/Dreamstalker-PRO-v1/Dreamstalker-PRO-v1.sch (KiCad schematic (older format))
At the start: 75 parts, among them J1 Header 2x3, J2 Header 2x5, J3 ST-033, J4 ATTEND_112J-TDAR-R01, M1 Vibration Motor, Q1 IRLML2402, Q2 BC807-40, Q3 BC807-40, Q4 BC807-40, Q5 BC807-40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

Commit message: Dreamstalker-PRO PCB improvements
Parts:
- removed U1: ATMEGA128L-8AI, Dreamstalker-Footprints:QFP80P1600X1600X120-64N, symbol Dreamstalker-Components:ATMEGA128L-8AI
- added C15: 10u, Dreamstalker-Footprints:CP_EIA-3216-18_Kemet-A, symbol Dreamstalker-Components:CP_Small
- added R24, R28, R30, R31: 100K, Dreamstalker-Footprints:R_0603_1608Metric, symbol Dreamstalker-Components:R_Small
- added U1: ATMEGA128L-8AU, Dreamstalker-Footprints:QFP80P1600X1600X120-64N, symbol Dreamstalker-Components:ATMEGA128L-8AU
- C13: value 0.1u -> 100n
- C16, C17, C18: value 1u -> 10n
- J1: value Header 2x3 -> UART Header
- J2: value Header 2x5 -> JTAG Header
- R17, R18, R27: value 10K -> 22
- R2: value 150 -> 0
- R3: value 47K -> 100K
- Y2: value 12.0 MHz -> 12.288M
Connections:
- net +3V: now also R2.2, U1.1 (~PEN), U1.21 (VCC_1), U1.52 (VCC_2), U1.64 (AVCC); no longer M1.1 (+), U3.24 (NC_6), U3.31 (NC_8), U3.5 (NC_1), U3.7 (NC_2)
- net DREQ: now also U1.14 ((OC0)_PB4)
- net GBUF: now also U1.59 (PF2_(ADC2))
- net GND: now also C15.2, R24.1, R28.1, R30.1, R31.1, U1.22 (GND_1), U1.53 (GND_2), U1.63 (GND_3); no longer U3.10 (GPIO3/SDATA), U3.11 (NC_3), U3.12 (NC_4), U3.25 (NC_7), U3.33 (SPIBOOT_/_GPIO0), U3.34 (GPIO1), U3.35 (NC_9), U3.36 (NC_10), U3.9 (GPIO2/DCLK)
- net HPTS: now also U1.4 ((XCK0/AIN0)_PE2)
- net IRRX: now also U1.61 (PF0_(ADC0))
- net IRTX: now also U1.35 (PC0_(A8))
- net KEY1: now also U1.29 ((ICP1)_PD4)
- net KEY2: now also U1.30 ((XCK1)_PD5)
- net KEY3: now also U1.25 ((SCL/INT0)_PD0)
- net KEY4: now also U1.26 ((SDA/INT1)_PD1)
- net KEY5: now also U1.31 ((T1)_PD6)
- net KEY6: now also U1.32 ((T2)_PD7)
- net LED1: now also U1.5 ((OC3A/AIN1)_PE3)
- net LED2: now also U1.6 ((OC3B/INT4)_PE4)
- net MGBUF: now also U1.33 (PG0(~WR))
- net MICP: now also U1.8 ((T3/INT6)_PE6)
- net MISO: now also U1.13 ((MISO)_PB3)
- net MLEFT: now also U1.34 (PG1(~RD))
- net MOSI: now also U1.12 ((MOSI)_PB2)
- net PDI: now also U1.2 (RXD0/(PDI)_PE0)
- net PDO: now also U1.3 ((TXD0/PDO)_PE1)
- net R1: now also U1.39 (PC4_(A12))
- net R2: now also U1.40 (PC5_(A13))
- net R3: now also U1.41 (PC6_(A14))
- net R4: now also U1.42 (PC7_(A15))
- net RESET: now also U1.20 (~RESET)
- net SCK: now also U1.11 ((SCK)_PB1)
- net SDCS: now also U1.10 ((~SS)_PB0)
- net SEGA: now also U1.51 (PA0_(AD0))
- net SEGB: now also U1.50 (PA1_(AD1))
- net SEGC: now also U1.49 (PA2_(AD2))
- net SEGD: now also U1.48 (PA3_(AD3))
- net SEGE: now also U1.47 (PA4_(AD4))
- net SEGF: now also U1.46 (PA5_(AD5))
- net SEGG: now also U1.45 (PA6_(AD6))
- net SEGH: now also U1.44 (PA7_(AD7))
- net SILENT: now also U1.37 (PC2_(A10))
- net SNDOFF: now also U1.7 ((OC3C/INT5)_PE5)
- net SOUND: now also U1.15 ((OC1A)_PB5)
- net TCK: now also U1.57 (PF4_(ADC4/TCK))
- net TDI: now also U1.54 (PF7_(ADC7/TDI))
- net TDO: now also U1.55 (PF6_(ADC6/TDO))
- net TMS: now also U1.56 (PF5_(ADC5/TMS))
- net TOSC1: now also U1.19 (TOSC1/PG4)
- net TOSC2: now also U1.18 (TOSC2/PG3)
- net VIBRO: now also Q1.1 (G), U1.36 (PC1_(A9)); no longer R2.1
- net XCS: now also U1.16 ((OC1B)_PB6)
- net XDCS: now also U1.17 ((OC2/OC1C)_PB7)
- net XRESET: now also U1.9 ((ICP3/INT7)_PE7)
- net at C7.1, C9.1, MK1.1 (P): now also R22.1; no longer R22.2
- net at C6.2, R20.2: now also R22.2, C15.1; no longer R22.1
- new net: R28.2, U3.10 (GPIO3/SDATA)
- new net: R31.2, U3.33 (SPIBOOT_/_GPIO0)
- new net: R30.2, U3.34 (GPIO1)
- new net: R24.2, U3.9 (GPIO2/DCLK)
- new net: M1.1 (+), R2.1
Other:
- moved on the sheet: C1, C10, C11, C12, C13, C14, C16, C17, C18, C2, C4, C5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

Commit message: Planned update
Parts:
- removed C6: 10u, Dreamstalker-Footprints:C_0805_2012Metric, symbol Dreamstalker-Components:C_Small
- added C19, C20: 10n, Dreamstalker-Footprints:C_0805_2012Metric, symbol Dreamstalker-Components:C_Small
- added C21: 0.1u, Dreamstalker-Footprints:C_0805_2012Metric, symbol Dreamstalker-Components:C_Small
- added C6: 10u, Dreamstalker-Footprints:CP_EIA-3216-18_Kemet-A, symbol Dreamstalker-Components:CP_Small
- added L1: L_Small, Dreamstalker-Footprints:L_0805_2012Metric, symbol Dreamstalker-Components:L_Small
- added R29, R32: 470, Dreamstalker-Footprints:R_0603_1608Metric, symbol Dreamstalker-Components:R_Small
- C13: value 100n -> 1u
- C17: value 10n -> 47n
- R17, R18: value 22 -> 20
- R2: value 0 -> 100
- R27: value 22 -> 10
- Y1: footprint Dreamstalker-Footprints:Crystal_C38-LF_D3.0mm_L8.0mm_Horizontal -> Dreamstalker-Footprints:Crystal_SMD_3215-2Pin_3.2x1.5mm
Connections:
- net +3V: now also L1.1; no longer U3.14 (DVDD1), U3.19 (DVDD2), U3.26 (RX), U3.32 (TEST), U3.38 (AVDD0), U3.43 (AVDD1), U3.45 (AVDD2), U3.6 (DVDD0)
- net GND: now also U3.11 (NC_3), U3.12 (NC_4), U3.25 (NC_7), U3.35 (NC_9), U3.36 (NC_10), C19.1, C20.2, C21.2
- net at U3.1 (MICP): now also C20.1, R29.2; no longer C7.2
- net at U3.2 (MICN): now also C19.2, R32.2; no longer C8.2
- net VSVDD: now reaches U3.24 (NC_6)
- net VSVDD: now also U3.14 (DVDD1), U3.19 (DVDD2), U3.26 (RX), U3.31 (NC_8), U3.32 (TEST), U3.38 (AVDD0), U3.43 (AVDD1), U3.45 (AVDD2), U3.5 (NC_1), U3.6 (DVDD0), U3.7 (NC_2), L1.2
- net at C15.1, R20.2, R22.2: now also C6.1
- net at R21.2, R23.1: now also C6.2
- net CD: now reaches J4.9 (DETECT)
- net CD: now also U1.38 (PC3_(A11))
- net AREF: now reaches U1.62 (AREF)
- net AREF: now also C21.1
- new net: C7.2, R29.1
- new net: C8.2, R32.1
Other:
- moved on the sheet: C1, C10, C11, C12, C14, C15, C16, C17, C18, C2, C4, C5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
