File: hardware/kicad/PRO/Dreamstalker-PRO-v2/Dreamstalker-PRO-v2.kicad_pcb (KiCad board)
At the start: 2 copper layers, 79 x 85 mm, 112 parts, among them J1 UART Header, J2 JTAG Header, J3 ST-033, J4 ATTEND_112J-TDAR-R01, J5 USB Power, J6 Li-Po 3.7V, M1 Vibration Motor, Q1 IRLML2402, Q2 BC807-40, Q3 BC807-40, Q4 BC807-40, Q5 BC807-40, Q6 KP-3216P3C, Q7 Si2333CDS, SW1 SELECT, SW2 ENTER, SW3 POWER, SW4 CHECK, SW5 [+], SW6 [-], U1 ATMEGA128L-8AI, U2 MC34119D, U3 VS1002D, U4 MCP73833, U5 RT9193-30PB, Y1 32768 KHz, Y2 12.288M

Commit message: Hardware: minor updates to kicad files
Parts:
- R36: value 470 -> 560
- R43: value 30K -> 75K
- R44: value 15K -> 33K
Connections:
- net /V_IN renamed V_IN
